File: hardware/LiveHacking.sch (KiCad schematic (older format))
At the start: 15 parts, among them J1 Conn_01x05, SW1 SW_Push, SW2 SW_Push, SW3 SW_Push, U1 Pico

Commit message: update project schmeatic start routing
Parts:
- added RN1, RN2: R_Pack04, Resistor_SMD:R_Array_Convex_4x0603, symbol Device:R_Pack04
- BT1: footprint (none) -> Badge-LiveHacking:12BH423GR; manf# (none) -> 12BH423-GR
- D1: footprint Diode_THT:D_DO-201AD_P15.24mm_Horizontal -> Diode_SMD:D_SOD-123F; manf# (none) -> MBR120LSFT3G
- D2, D3, D4, D5, D6, D7, D8, D9: footprint (none) -> Badge-LiveHacking:LYT77K-K2M1-NoHole; manf# (none) -> AA3528SECKT/J309
- J1: footprint (none) -> Connector_PinHeader_2.54mm:PinHeader_1x05_P2.54mm_Vertical
- SW1: value SW_Push -> RST; footprint (none) -> Button_Switch_SMD:SW_SPST_TL3342
- SW2, SW3: footprint (none) -> Button_Switch_SMD:SW_SPST_TL3342
- U1: footprint RPi_Pico:RPi_Pico_SMD_TH -> Badge-LiveHacking:RPi_Pico_SMD_TH; symbol MCU_RaspberryPi_and_Boards:Pico -> LiveHacking-rescue:Pico-MCU_RaspberryPi_and_Boards
Connections:
- net BTN1: now also U1.17 (GPIO13); no longer U1.16 (GPIO12)
- net BTN2: now also U1.16 (GPIO12); no longer U1.17 (GPIO13)
- net GND: now also RN1.1 (R1.1), RN1.2 (R2.1), RN1.3 (R3.1), RN1.4 (R4.1), RN2.1 (R1.1), RN2.2 (R2.1), RN2.3 (R3.1), RN2.4 (R4.1); no longer D2.1 (K), D3.1 (K), D4.1 (K), D5.1 (K), D6.1 (K), D7.1 (K), D8.1 (K), D9.1 (K)
- new net: D2.1 (K), RN1.8 (R1.2)
- new net: D3.1 (K), RN1.7 (R2.2)
- new net: D7.1 (K), RN2.8 (R1.2)
- new net: D9.1 (K), RN2.7 (R2.2)
- new net: D5.1 (K), RN1.6 (R3.2)
- new net: D4.1 (K), RN1.5 (R4.2)
- new net: D8.1 (K), RN2.6 (R3.2)
- new net: D6.1 (K), RN2.5 (R4.2)
Other:
- moved on the sheet: D6, D7, D8, D9
